File: Bk scheda led e pulsanti 1_2.kicad_pcb (KiCad board)
At the start: 2 copper layers, 262 x 120 mm, 187 parts, among them J35 Screw_Terminal_01x02, J36 Screw_Terminal_01x16, J37 Screw_Terminal_01x16, SW1 SW_SPDT_MSM, SW10 SW_SPDT_MSM, SW11 SW_SPDT_MSM, SW12 SW_SPDT_MSM, SW13 SW_SPDT_MSM, SW14 SW_SPDT_MSM, SW15 SW_SPDT_MSM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

Commit message: Modifica intitolazione su PCB
Other:
- board text added: "G.R. - D.L. - DIP. ELETTRONICA - ISIS BASSA FRIULANA - 2025/26"
- board text removed: "G.R. - D.L. - ISIS BASSA FRIULANA - 2025/26"
Changed lines of the file:
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@@
 			(plot_on_all_layers_selection 0x00000000_00000000_00000000_00000000)
 			(disableapertmacros no)
-			(usegerberextensions no)
+			(usegerberextensions yes)
 			(usegerberattributes yes)
 			(usegerberadvancedattributes yes)
-			(creategerberjobfile yes)
+			(creategerberjobfile no)
 			(dashed_line_dash_ratio 12.000000)
 			(dashed_line_gap_ratio 3.000000)
@@
 			(drillshape 0)
 			(scaleselection 1)
-			(outputdirectory "D:/KiCad/Traccia stampati/SImulatore Beckhoff1.8/")
+			(outputdirectory "Gerber/")
 		)
 	)
@@
 		)
 	)
-	(gr_text "G.R. - D.L. - ISIS BASSA FRIULANA - 2025/26"
+	(gr_text "G.R. - D.L. - DIP. ELETTRONICA - ISIS BASSA FRIULANA - 2025/26"
 		(at 148.5 107.8 0)
 		(layer "B.SilkS")
